File: main/mu100-dit.kicad_pcb (KiCad board)
At the start: 2 copper layers, 17.6 x 40 mm, 22 parts, among them J1 Conn_01x10_Female, J2 Conn_01x02_Male, U1 TOTX-177L, U2 AK4103A, U3 APX809S-46SR-7

Commit message: WIP
Parts:
- C4, R1, R2: moved to F.Cu
- moved R1 1.26 mm to (84.8, 86.5), turned to 0 degrees
- moved C4 1.08 mm to (84.8, 84.1)
- moved R2 0.89 mm to (84.8, 81.7)
- moved J2 0.40 mm to (80.5, 85.7)
- moved JP1 0.10 mm to (85.2, 100.8)
- moved JP2 0.10 mm to (85.2, 103.1)
- moved JP3 0.10 mm to (85.2, 105.4)
- moved JP4 0.10 mm to (85.2, 107.7)
- moved JP9 0.10 mm to (85.2, 110.0)
Routing:
- net GND: track 52.2 -> 73.6 mm, vias 8 -> 20
- net /TXP: track 24.9 -> 27.9 mm, vias 0 -> 1
- net +5V: track 85.0 -> 87.9 mm
- net Net-(C4-Pad1): track 5.93 -> 4.63 mm
- net Net-(C4-Pad2): track 2.63 -> 3.51 mm
- net /FS1: track 8.49 -> 7.92 mm
Other:
- board size 17.6 x 40 mm -> 18 x 40 mm
- board text added: "Coax"
- board text removed: "Coax (OPT.)"
