File: main/mu100-dit.kicad_sch (KiCad schematic)
At the start: 22 parts, among them J1 Conn_01x10_Female, J2 Conn_01x02_Male, U1 TOTX-177L, U2 AK4103A, U3 APX809S-46SR-7

Commit message: Unground mounting holes, rearrange DIF0/DIF1 vias to avoid bridge
Parts:
- removed H1, H2: MountingHole_Pad, MountingHole:MountingHole_3.2mm_M3_ISO7380_Pad_TopBottom, symbol Mechanical:MountingHole_Pad
Changed lines of the file:
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@@
   (junction (at 103.505 123.825) (diameter 0) (color 0 0 0 0)
-  )
-  (junction (at 139.065 145.415) (diameter 0) (color 0 0 0 0)
   )
   (junction (at 103.505 126.365) (diameter 0) (color 0 0 0 0)
@@
     (stroke (width 0) (type default) (color 0 0 0 0))
   )
-  (wire (pts (xy 139.065 145.415) (xy 142.24 145.415))
-    (stroke (width 0) (type default) (color 0 0 0 0))
-  )
   (wire (pts (xy 187.96 83.185) (xy 197.485 83.185))
     (stroke (width 0) (type default) (color 0 0 0 0))
@@
   (wire (pts (xy 112.395 131.445) (xy 121.285 131.445))
     (stroke (width 0) (type solid) (color 0 0 0 0))
-  )
-  (wire (pts (xy 135.255 145.415) (xy 139.065 145.415))
-    (stroke (width 0) (type default) (color 0 0 0 0))
   )
   (wire (pts (xy 55.88 127) (xy 58.42 127))
@@
     (pin "2")
   )
-  (symbol (lib_id "Mechanical:MountingHole_Pad") (at 142.24 142.875 0) (unit 1)
-    (in_bom yes) (on_board yes) (fields_autoplaced)
-    (property "Reference" "H2" (id 0) (at 145.415 140.3349 0)
-      (effects (font (size 1.27 1.27)) (justify left))
-    )
-    (property "Value" "MountingHole_Pad" (id 1) (at 145.415 142.8749 0)
-      (effects (font (size 1.27 1.27)) (justify left))
-    )
-    (property "Footprint" "MountingHole:MountingHole_3.2mm_M3_ISO7380_Pad_TopBottom" (id 2) (at 142.24 142.875 0)
-      (effects (font (size 1.27 1.27)) hide)
-    )
-    (property "Datasheet" "~" (id 3) (at 142.24 142.875 0)
-      (effects (font (size 1.27 1.27)) hide)
-    )
-    (pin "1")
-  )
   (symbol (lib_id "power:GND") (at 172.72 90.805 90) (unit 1)
     (in_bom yes) (on_board yes)
@@
     )
     (property "Datasheet" "" (id 3) (at 156.845 103.505 0)
-      (effects (font (size 1.27 1.27)) hide)
-    )
-    (pin "1")
-  )
-  (symbol (lib_id "Mechanical:MountingHole_Pad") (at 135.255 142.875 0) (unit 1)
-    (in_bom yes) (on_board yes)
-    (property "Reference" "H1" (id 0) (at 130.175 140.335 0)
-      (effects (font (size 1.27 1.27)) (justify left))
-    )
-    (property "Value" "MountingHole_Pad" (id 1) (at 115.57 142.875 0)
-      (effects (font (size 1.27 1.27)) (justify left))
-    )
-    (property "Footprint" "MountingHole:MountingHole_3.2mm_M3_ISO7380_Pad_TopBottom" (id 2) (at 135.255 142.875 0)
-      (effects (font (size 1.27 1.27)) hide)
-    )
-    (property "Datasheet" "~" (id 3) (at 135.255 142.875 0)
       (effects (font (size 1.27 1.27)) hide)
     )
@@
     (pin "1")
   )
-  (symbol (lib_id "power:GND") (at 139.065 145.415 0) (unit 1)
-    (in_bom yes) (on_board yes) (fields_autoplaced)
-    (property "Reference" "#PWR0113" (id 0) (at 139.065 151.765 0)
-      (effects (font (size 1.27 1.27)) hide)
-    )
-    (property "Value" "GND" (id 1) (at 139.065 150.495 0))
-    (property "Footprint" "" (id 2) (at 139.065 145.415 0)
-      (effects (font (size 1.27 1.27)) hide)
-    )
-    (property "Datasheet" "" (id 3) (at 139.065 145.415 0)
-      (effects (font (size 1.27 1.27)) hide)
-    )
-    (pin "1")
-  )
   (symbol (lib_id "Device:R_Small_US") (at 200.025 121.285 180) (unit 1)
     (in_bom yes) (on_board yes)
@@
       (reference "#PWR0112") (unit 1) (value "GND") (footprint "")
     )
-    (path "/62399e8a-c65f-4f54-a12d-9987c4d2db9e"
-      (reference "#PWR0113") (unit 1) (value "GND") (footprint "")
-    )
     (path "/73976c76-6e85-44ac-a6e4-c1b2c52a8b22"
       (reference "#PWR0114") (unit 1) (value "GND") (footprint "")
@@
       (reference "C4") (unit 1) (value "0.1uF") (footprint "Capacitor_SMD:C_0805_2012Metric_Pad1.18x1.45mm_HandSolder")
     )
-    (path "/296f96cb-3a0e-4d9e-a759-384daaf57c05"
-      (reference "H1") (unit 1) (value "MountingHole_Pad") (footprint "MountingHole:MountingHole_3.2mm_M3_ISO7380_Pad_TopBottom")
-    )
-    (path "/1db16de4-511f-4d18-a697-e02c9e9ae0f3"
-      (reference "H2") (unit 1) (value "MountingHole_Pad") (footprint "MountingHole:MountingHole_3.2mm_M3_ISO7380_Pad_TopBottom")
-    )
     (path "/01106a52-6b7d-40fd-b165-c927be1f6a1d"

Commit message: minor tweaks to main board
Connections:
- net GND: now also J1.1 (Pin_1)
- no-connect marks 5 -> 4
Changed lines of the file:
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@@
   (junction (at 58.42 127) (diameter 0) (color 0 0 0 0)
   )
+  (junction (at 81.28 88.9) (diameter 0) (color 0 0 0 0)
+  )
   (junction (at 67.945 93.98) (diameter 0) (color 0 0 0 0)
   )
@@
   )
   (no_connect (at 121.285 116.205))
-  (no_connect (at 87.63 83.82))
   (no_connect (at 156.845 108.585))
   (no_connect (at 156.845 126.365))
   (no_connect (at 156.845 98.425))
+  (wire (pts (xy 87.63 83.82) (xy 81.28 83.82))
+    (stroke (width 0) (type default) (color 0 0 0 0))
+  )
   (wire (pts (xy 63.5 86.36) (xy 67.945 86.36))
     (stroke (width 0) (type default) (color 0 0 0 0))
@@
     (stroke (width 0) (type default) (color 0 0 0 0))
   )
+  (wire (pts (xy 81.28 88.9) (xy 87.63 88.9))
+    (stroke (width 0) (type default) (color 0 0 0 0))
+  )
   (wire (pts (xy 156.845 121.285) (xy 167.005 121.285))
     (stroke (width 0) (type solid) (color 0 0 0 0))
@@
     (stroke (width 0) (type solid) (color 0 0 0 0))
   )
+  (wire (pts (xy 81.28 83.82) (xy 81.28 88.9))
+    (stroke (width 0) (type default) (color 0 0 0 0))
+  )
   (wire (pts (xy 55.88 127) (xy 58.42 127))
     (stroke (width 0) (type default) (color 0 0 0 0))
@@
     (stroke (width 0) (type default) (color 0 0 0 0))
   )
-  (wire (pts (xy 67.945 88.9) (xy 87.63 88.9))
-    (stroke (width 0) (type default) (color 0 0 0 0))
-  )
+  (wire (pts (xy 67.945 88.9) (xy 81.28 88.9))
+    (stroke (width 0) (type default) (color 0 0 0 0))
+  )
