File: main/mu100-dit.kicad_sch (KiCad schematic)
At the start: 20 parts, among them J1 Conn_01x10_Female, J2 Conn_01x02_Male, U1 TOTX-177L, U2 AK4103A, U3 APX809S-46SR-7

Commit message: FInal board revision
Connections:
- net GND: no longer J1.1 (Pin_1)
- no-connect marks 4 -> 5
Changed lines of the file:
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@@
   (junction (at 58.42 127) (diameter 0) (color 0 0 0 0)
-  )
-  (junction (at 81.28 88.9) (diameter 0) (color 0 0 0 0)
   )
   (junction (at 67.945 93.98) (diameter 0) (color 0 0 0 0)
@@
   (no_connect (at 156.845 108.585))
   (no_connect (at 156.845 126.365))
+  (no_connect (at 87.63 83.82))
   (no_connect (at 156.845 98.425))
-  (wire (pts (xy 87.63 83.82) (xy 81.28 83.82))
-    (stroke (width 0) (type default) (color 0 0 0 0))
-  )
   (wire (pts (xy 63.5 86.36) (xy 67.945 86.36))
     (stroke (width 0) (type default) (color 0 0 0 0))
@@
     (stroke (width 0) (type default) (color 0 0 0 0))
   )
-  (wire (pts (xy 81.28 88.9) (xy 87.63 88.9))
+  (wire (pts (xy 67.945 88.9) (xy 87.63 88.9))
     (stroke (width 0) (type default) (color 0 0 0 0))
   )
@@
     (stroke (width 0) (type solid) (color 0 0 0 0))
   )
-  (wire (pts (xy 81.28 83.82) (xy 81.28 88.9))
-    (stroke (width 0) (type default) (color 0 0 0 0))
-  )
   (wire (pts (xy 55.88 127) (xy 58.42 127))
     (stroke (width 0) (type default) (color 0 0 0 0))
@@
     (stroke (width 0) (type default) (color 0 0 0 0))
   )
-  (wire (pts (xy 67.945 88.9) (xy 81.28 88.9))
-    (stroke (width 0) (type default) (color 0 0 0 0))
-  )
