File: main/other-board-revisions/rearrange/mu100-dit.kicad_pcb (KiCad board)
At the start: 2 copper layers, 18 x 40 mm, 22 parts, among them J1 Conn_01x10_Female, J2 Conn_01x02_Male, U1 TOTX-177L, U2 AK4103A, U3 APX809S-46SR-7

Commit message: FInal board revision
Parts:
- moved R2 36.6 mm to (85.3, 118.3)
- moved C4 31.8 mm to (85.3, 115.9)
- moved C3 30.9 mm to (81.8, 86.3)
- moved U3 30.9 mm to (81.8, 82.8)
- moved J2 29.4 mm to (80.1, 115.0), turned to 0 degrees
- moved R1 27.1 mm to (85.3, 113.5)
- moved JP9 5.58 mm to (90.7, 108.9)
- moved JP8 1.15 mm to (90.7, 111.2)
Routing:
- net /RESET: track 12.5 -> 45.1 mm
- net GND: track 73.6 -> 48.7 mm, vias 16 -> 11
- net +5V: track 88.3 -> 81.3 mm
- net /CKS1: track 8.50 -> 1.97 mm
- net Net-(C4-Pad1): track 4.63 -> 0.28 mm
- net Net-(C4-Pad2): track 3.51 -> 0.00 mm
- net /TXP: track 27.9 -> 28.6 mm, vias 1 -> 2
Other:
- board text removed: "v1.1"
